File: hardware/01_SNES_BUS_AND_CIC.kicad_sch (KiCad schematic)
At the start: 0 parts

Commit message: feat: complete KiCad schematics with real components, translate repo to English
- Rewritten generate_schematics.py (2236 lines) with real KiCad library refs
- 62 components placed across 5 schematic sheets + root
- Physical wires connecting all power pins, decoupling caps, crystal, USB
- Custom symbols: RP2350B, ESP32-C6-MINI, SY8089, SNES_62PIN, SST39VF040
- Translated all documentation from Portuguese to English
- Updated author to forg3
- Added docs/pin-mapping.md with complete 62-pin SNES connector mapping
- All 6 .kicad_sch files validated (balanced parens, 62 components total)

Author: forg3
Parts:
- added C5: 100nF, Capacitor_SMD:C_0402_1005Metric, symbol Device:C
- added D1, D2: USBLC6-2SC6, Package_TO_SOT_SMD:SOT-23-6_Handsoldering, symbol Custom:USBLC6-2SC6
- added P1: SNES_EDGE_62, Connector_CardEdge:SNES_CartridgeEdge_62Pin_2.50mm, symbol Custom:SNES_62PIN
- added U1: PIC12F629-I/SN, Package_SO:SOIC-8_3.9x4.9mm_P1.27mm, symbol MCU_Microchip_PIC:PIC12F629
Other:
- note added: "SHEET 1: SNES 62-Pin Cartridge Connector & SuperCIC\nPitch: 2.50mm Metric | PCB: 1.20mm ENIG 30-deg Bevel\n\nU1: PIC12F629 SuperCIC (NTSC/PAL auto-detect)\nD1,D2: USBLC6-2SC6 ESD/TVS protection\nC5: 100nF decoupling"
- note removed: "SHEET 1: SNES 62-PIN CARTRIDGE CONNECTOR & SUPERCIC Pinout Specifications: - Pitch: 2.50mm Metric Pitch (DO NOT USE 2.54mm!) - PCB Thickness: 1.20mm ENIG with 30-degree Beveling Signals: - Power: Pins 27, 58 = +5V_SNES, Pins 5, 36 = GND - Data: Pins 19-22 = SNES_D0..SNES_D3, Pins 50-53 = SNES_D4..SNES_D7 - Address: Pins 17..6 = SNES_A0..SNES_A11, Pins 37..40 = SNES_A12..SNES_A15 - Bank Address: P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"
