File: hardware/02_LEVEL_SHIFTERS_AND_FLASH.kicad_sch (KiCad schematic)
At the start: 0 parts

Commit message: feat: complete KiCad schematics with real components, translate repo to English
- Rewritten generate_schematics.py (2236 lines) with real KiCad library refs
- 62 components placed across 5 schematic sheets + root
- Physical wires connecting all power pins, decoupling caps, crystal, USB
- Custom symbols: RP2350B, ESP32-C6-MINI, SY8089, SNES_62PIN, SST39VF040
- Translated all documentation from Portuguese to English
- Updated author to forg3
- Added docs/pin-mapping.md with complete 62-pin SNES connector mapping
- All 6 .kicad_sch files validated (balanced parens, 62 components total)

Author: forg3
Parts:
- added C6, C7, C8, C9: 100nF, Capacitor_SMD:C_0402_1005Metric, symbol Device:C
- added R7: 10k, Resistor_SMD:R_0402_1005Metric, symbol Device:R
- added U2, U3: 74LVC541APW, Package_SO:TSSOP-20_4.4x6.5mm_P0.65mm, symbol Logic_74xx:74LVC541A
- added U4: SN74LVC8T245PWR, Package_SO:TSSOP-24_4.4x7.8mm_P0.65mm, symbol Logic_74xx:SN74LVC8T245PWR
- added U5: SST39VF040-70-4C-WHE, Package_SO:TSOP-32_8x14mm_P0.5mm, symbol Custom:SST39VF040
Connections:
- new net BUS_A11: U5.5 (A4)
Other:
- note added: "SHEET 2: Voltage Level Shifters & Boot Flash ROM\n\nU2,U3: 74LVC541APW (5V->3.3V Address/Control)\nU4: SN74LVC8T245PWR (Bidir Data Bus 5V<->3.3V)\nU5: SST39VF040 512KB Parallel NOR Flash\nR7: 10k pull-up (Flash /WE HW write-protect)\nC6-C9: 100nF decoupling per IC"
- note removed: "SHEET 2: VOLTAGE LEVEL SHIFTERS & BOOT FLASH ROM Level Shifting Architecture (5V TTL <-> 3.3V CMOS): 1. Address & Control Bus (SNES -> Cartridge, Unidirectional 5V -> 3.3V): - U2: 74LVC541APW (TSSOP-20) for SNES_A0..SNES_A7, /RD, /WR - U3: 74LVC541APW (TSSOP-20) for SNES_A8..SNES_A15, /ROMSEL, PHI2 - Inputs are 5V tolerant when powered at 3.3V. Propagation delay: ~3.0 ns - /OE1, /OE2 tied to GND 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"
