File: hardware/03_RP2350_SUBSYSTEM.kicad_sch (KiCad schematic)
At the start: 0 parts

Commit message: feat: complete KiCad schematics with real components, translate repo to English
- Rewritten generate_schematics.py (2236 lines) with real KiCad library refs
- 62 components placed across 5 schematic sheets + root
- Physical wires connecting all power pins, decoupling caps, crystal, USB
- Custom symbols: RP2350B, ESP32-C6-MINI, SY8089, SNES_62PIN, SST39VF040
- Translated all documentation from Portuguese to English
- Updated author to forg3
- Added docs/pin-mapping.md with complete 62-pin SNES connector mapping
- All 6 .kicad_sch files validated (balanced parens, 62 components total)

Author: forg3
Parts:
- added C10, C11: 15pF, Capacitor_SMD:C_0402_1005Metric, symbol Device:C
- added C12, C13, C18: 100nF, Capacitor_SMD:C_0402_1005Metric, symbol Device:C
- added C17: 10uF, Capacitor_SMD:C_0805_2012Metric, symbol Device:C
- added J1: TYPE-C-31-M-12, Connector_USB:USB_C_Receptacle_HRO_TYPE-C-31-M-12, symbol Connector:USB_C_Receptacle_16P
- added R3, R4: 5.1k, Resistor_SMD:R_0402_1005Metric, symbol Device:R
- added R5, R6: 27R, Resistor_SMD:R_0402_1005Metric, symbol Device:R
- added R8: 10k, Resistor_SMD:R_0402_1005Metric, symbol Device:R
- added SW1: BOOTSEL, Button_Switch_SMD:SW_SPST_TL3342, symbol Device:SW_Push
- added SW2: RESET, Button_Switch_SMD:SW_SPST_TL3342, symbol Device:SW_Push
- added U6: RP2350B, Package_DFN_QFN:QFN-80-1EP_10x10mm_P0.5mm_EP6.1x6.1mm, symbol Custom:RP2350B
- added U7: W25Q128JVSIQ, Package_SO:SOIC-8_3.9x4.9mm_P1.27mm, symbol Memory_Flash:W25Q128
- added Y1: 12.000MHz, Crystal:Crystal_SMD_3215-2Pin_3.2x1.5mm, symbol Device:Crystal
Connections:
- new net: C12.2, C13.1
Other:
- note added: "SHEET 3: RP2350B Dual-Core MCU Subsystem\n\nU6: RP2350B (Cortex-M33 x2, 520KB SRAM)\nU7: W25Q128JVSIQ 16MB QSPI Flash\nY1: 12MHz crystal + 15pF load caps\nJ1: USB-C (UF2 drag-and-drop)\nSW1: BOOTSEL, SW2: RESET\nR3-R4: 5.1k USB-C CC pulldowns\nR5-R6: 27R USB series resistors\nR8: 10k QSPI CS pull-up"
- note removed: "SHEET 3: RP2350B DUAL-CORE MCU SUBSYSTEM MCU Selection: Raspberry Pi RP2350B (QFN-80) - 48 GPIOs allow dedicated bus taps and rich peripheral connectivity - Dual ARM Cortex-M33 cores @ 150MHz (overclockable to 250MHz+) - 520KB on-chip SRAM: perfectly hosts the Home Assistant Mailbox & dynamic snapshot - 12 PIO State Machines for real-time bus interception, cycle-accurate timing Pin Allocation: - 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"
