File: hardware/04_ESP32C6_WIFI_IOT.kicad_sch (KiCad schematic)
At the start: 0 parts

Commit message: feat: complete KiCad schematics with real components, translate repo to English
- Rewritten generate_schematics.py (2236 lines) with real KiCad library refs
- 62 components placed across 5 schematic sheets + root
- Physical wires connecting all power pins, decoupling caps, crystal, USB
- Custom symbols: RP2350B, ESP32-C6-MINI, SY8089, SNES_62PIN, SST39VF040
- Translated all documentation from Portuguese to English
- Updated author to forg3
- Added docs/pin-mapping.md with complete 62-pin SNES connector mapping
- All 6 .kicad_sch files validated (balanced parens, 62 components total)

Author: forg3
Parts:
- added C14: 100nF, Capacitor_SMD:C_0402_1005Metric, symbol Device:C
- added C15: 10uF, Capacitor_SMD:C_0805_2012Metric, symbol Device:C
- added D3: WS2812B-2020, LED_SMD:LED_WS2812B_PLCC4_3.2x3.2mm_P1.75mm, symbol Custom:WS2812B
- added R10, R9: 10k, Resistor_SMD:R_0402_1005Metric, symbol Device:R
- added SW3: ESP_BOOT, Button_Switch_SMD:SW_SPST_TL3342, symbol Device:SW_Push
- added SW4: ESP_EN, Button_Switch_SMD:SW_SPST_TL3342, symbol Device:SW_Push
- added U8: ESP32-C6-MINI-1-N4, RF_Module:ESP32-C6-MINI-1, symbol Custom:ESP32-C6-MINI-1
Other:
- note added: "SHEET 4: ESP32-C6 Wi-Fi 6 / BLE / Thread Coprocessor\n\nU8: ESP32-C6-MINI-1-N4\n Wi-Fi 6, BLE 5, 802.15.4 (Thread/Zigbee)\nD3: WS2812B RGB status LED\nSW3: ESP_BOOT, SW4: ESP_EN\nR9,R10: 10k pull-ups\nC14: 100nF, C15: 10uF decoupling"
- note removed: "SHEET 4: ESP32-C6 WI-FI 6 / BLE / THREAD COPROCESSOR Module: Espressif ESP32-C6-MINI-1 (or ESP32-C6-WROOM-1) - 32-bit RISC-V single-core @ 160MHz, 512KB SRAM, 4MB/8MB Flash - Wi-Fi 6 (2.4 GHz 802.11ax), Bluetooth 5 (LE), IEEE 802.15.4 (Thread/Zigbee) - Built-in certified PCB antenna (placed at the top edge of cartridge with keepout) Role in SNES Smart Home: - Connects to local Wi-Fi and establish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"
