File: hardware/05_PERIPHERALS_AND_POWER.kicad_sch (KiCad schematic)
At the start: 0 parts

Commit message: feat: complete KiCad schematics with real components, translate repo to English
- Rewritten generate_schematics.py (2236 lines) with real KiCad library refs
- 62 components placed across 5 schematic sheets + root
- Physical wires connecting all power pins, decoupling caps, crystal, USB
- Custom symbols: RP2350B, ESP32-C6-MINI, SY8089, SNES_62PIN, SST39VF040
- Translated all documentation from Portuguese to English
- Updated author to forg3
- Added docs/pin-mapping.md with complete 62-pin SNES connector mapping
- All 6 .kicad_sch files validated (balanced parens, 62 components total)

Author: forg3
Parts:
- added BT1: CR1220, Battery:BatteryHolder_CR1220_Holder, symbol Battery:BatteryHolder_CR1220
- added C1, C4: 47uF, Capacitor_SMD:C_1206_3216Metric, symbol Device:C
- added C2, C3: 22uF, Capacitor_SMD:C_0805_2012Metric, symbol Device:C
- added D4: SS34, Diode_SMD:D_SMA, symbol Device:D
- added F1: 1206L150PR, Fuse:Fuse_1206_3216Metric, symbol Device:Polyfuse
- added J4: TF-01A, Connector_Card:TF_TF-01A, symbol Connector:Conn_01x09_Pin
- added J5: KF2EDG-3.5-3P, TerminalBlock:TerminalBlock_bornier-3_P5.08mm, symbol Connector:Conn_01x03_Pin
- added J6: JST_SH_1.0mm_4P, Connector_JST:JST_SH_SM04B-SRSS-TB_1.00mm, symbol Connector:Conn_01x04_Pin
- added L1: 2.2uH, Inductor_SMD:L_0805_2012Metric, symbol Device:L
- added R1: 100k, Resistor_SMD:R_0402_1005Metric, symbol Device:R
- added R11, R12: 4.7k, Resistor_SMD:R_0402_1005Metric, symbol Device:R
- added R13, R14, R16, R17: 10k, Resistor_SMD:R_0402_1005Metric, symbol Device:R
- added R15: 120R, Resistor_SMD:R_0603_1608Metric, symbol Device:R
- added R2: 22k, Resistor_SMD:R_0402_1005Metric, symbol Device:R
- added U10: DS3231MZ+, Package_SO:SOIC-8_3.9x4.9mm_P1.27mm, symbol Timer_RTC:DS3231
- added U11: MAX3485, Package_SO:SOIC-8_3.9x4.9mm_P1.27mm, symbol Interface_UART:MAX3485
- added U9: SY8089AAAC, Package_TO_SOT_SMD:SOT-23-5_Handsoldering, symbol Custom:SY8089
Connections:
- new net +5V_PROT: U9.1 (VIN)
- new net FB: R1.1, U9.5 (FB)
- new net RS485_A: R15.1
Other:
- note added: "SHEET 5: Peripherals & 5V->3.3V Power Supply\n\nU9: SY8089AAAC Buck 5V->3.3V 2.0A (>92% eff)\nU10: DS3231MZ+ RTC (+-5ppm, battery backup)\nU11: MAX3485 RS-485 Transceiver\nD4: SS34 Schottky (reverse polarity)\nF1: PTC 1.5A (overcurrent)\nL1: 2.2uH inductor\nBT1: CR1220 battery holder"
- note removed: "SHEET 5: PERIPHERALS (MICROSD, RTC, RS-485, I2C) & 5V->3.3V BUCK 1. Power Supply Subsystem (High Efficiency Synchronous Buck): - Input: +5V_SNES from cartridge edge (pins 27, 58) - Reverse polarity / overcurrent protection: SS34 Schottky diode / PTC resettable fuse (1.5A) - U9: Silergy SY8089AAAC (or AP62200 / TPS62088) Synchronous Step-Down DC-DC Converter Package: SOT-23-5, 1.5MHz switching fre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"
