File: hardware/snes_smarthome_cartridge.kicad_sch (KiCad schematic)
At the start: 0 parts

Commit message: feat: complete KiCad schematics with real components, translate repo to English
- Rewritten generate_schematics.py (2236 lines) with real KiCad library refs
- 62 components placed across 5 schematic sheets + root
- Physical wires connecting all power pins, decoupling caps, crystal, USB
- Custom symbols: RP2350B, ESP32-C6-MINI, SY8089, SNES_62PIN, SST39VF040
- Translated all documentation from Portuguese to English
- Updated author to forg3
- Added docs/pin-mapping.md with complete 62-pin SNES connector mapping
- All 6 .kicad_sch files validated (balanced parens, 62 components total)

Author: forg3
Other:
- sheet 01_SNES_BUS_AND_CIC ports: added /IRQ, /RD, /RESET, /ROMSEL, /WR, CIC_CLK, CIC_DAT1, CIC_DAT2, CIC_RST, PHI2, SNES_A0, SNES_A1, SNES_A10, SNES_A11, SNES_A12, SNES_A13, SNES_A14, SNES_A15, SNES_A16, SNES_A17, SNES_A18, SNES_A19, SNES_A2, SNES_A20, SNES_A21, SNES_A22, SNES_A23, SNES_A3, SNES_A4, SNES_A5, SNES_A6, SNES_A7, SNES_A8, SNES_A9, SNES_D0, SNES_D1, SNES_D2, SNES_D3, SNES_D4, SNES_D5, SNES_D6, SNES_D7; removed none
- sheet 02_LEVEL_SHIFTERS_AND_FLASH ports: added /RD, /ROMSEL, /WR, BUS_A0, BUS_A1, BUS_A10, BUS_A11, BUS_A12, BUS_A13, BUS_A14, BUS_A15, BUS_A2, BUS_A3, BUS_A4, BUS_A5, BUS_A6, BUS_A7, BUS_A8, BUS_A9, BUS_D0, BUS_D1, BUS_D2, BUS_D3, BUS_D4, BUS_D5, BUS_D6, BUS_D7, BUS_PHI2, BUS_RD, BUS_ROMSEL, BUS_WR, PHI2, SNES_A0, SNES_A1, SNES_A10, SNES_A11, SNES_A12, SNES_A13, SNES_A14, SNES_A15, SNES_A2, SNES_A3, SNES_A4, SNES_A5, SNES_A6, SNES_A7, SNES_A8, SNES_A9, SNES_D0, SNES_D1, SNES_D2, SNES_D3, SNES_D4, SNES_D5, SNES_D6, SNES_D7; removed none
- sheet 03_RP2350_SUBSYSTEM ports: added BUS_A0, BUS_A1, BUS_A10, BUS_A11, BUS_A12, BUS_A13, BUS_A14, BUS_A15, BUS_A2, BUS_A3, BUS_A4, BUS_A5, BUS_A6, BUS_A7, BUS_A8, BUS_A9, BUS_D0, BUS_D1, BUS_D2, BUS_D3, BUS_D4, BUS_D5, BUS_D6, BUS_D7, BUS_PHI2, BUS_RD, BUS_ROMSEL, BUS_WR, ESP_INT, I2C_SCL, I2C_SDA, JUMP_BOOTSEL, JUMP_RST, LED_HEARTBEAT, LED_STATUS, LED_WIFI, RS485_RX, RS485_TX, SD_CS, SD_MISO, SD_MOSI, SD_SCK, SPI_CS, SPI_MISO, SPI_MOSI, SPI_SCK, UART_RX, UART_TX; removed none
- sheet 04_ESP32C6_WIFI_IOT ports: added ESP_INT, SPI_CS, SPI_MISO, SPI_MOSI, SPI_SCK, UART_RX, UART_TX; removed none
- sheet 05_PERIPHERALS_AND_POWER ports: added I2C_SCL, I2C_SDA, LED_HEARTBEAT, LED_STATUS, LED_WIFI, RS485_RX, RS485_TX, SD_CS, SD_MISO, SD_MOSI, SD_SCK; removed none
- note added: "SUPER FAMICOM / SNES SMART HOME INTERFACE CARTRIDGE V1.0\n\nSystem Overview:\n- Sheet 1: 62-Pin SNES Bus Edge Connector (2.50mm pitch) + SuperCIC PIC12F629\n- Sheet 2: 74LVC541 + SN74LVC8T245 Level Shifters + 4Mbit Parallel Boot Flash\n- Sheet 3: RP2350B MCU Subsystem (Dual Cortex-M33, Mailbox, 16MB QSPI, USB-C)\n- Sheet 4: ESP32-C6-MINI-1 Wi-Fi 6 / BLE / Thread (Home Assistant REST/WS)\n- Sheet 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"
- note removed: "SUPER FAMICOM / SNES SMART HOME INTERFACE CARTRIDGE V1.0 System Overview: - Sheet 1: 62-Pin SNES Bus Edge Connector (2.50mm pitch, 1.2mm PCB) + SuperCIC PIC12F629 - Sheet 2: 74LVC541 + SN74LVC8T245 Level Shifters + 4Mbit Parallel Boot Flash (SST39VF040) - Sheet 3: RP2350B MCU Subsystem (Dual Cortex-M33, 520KB SRAM Mailbox, 16MB QSPI, USB-C) - Sheet 4: ESP32-C6-MINI-1 Wi-Fi 6 / BLE / 802.15.4 Modu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"
